File: ETI Polysynth.sch (KiCad schematic (older format))
At the start: 0 parts

Commit message: WIP
Parts:
- added U? (x2): 74LS266, symbol 74xx_IEEE:74LS266
- added U? (x2): 74LS08, symbol 74xx:74LS08
- added U? (x5): 74LS32, symbol 74xx:74LS32
- added U? (x5): 74LS04, symbol 74xx:74LS04
- added U?: 74LS00, symbol 74xx:74LS00
- added U? (x2): 74LS74, symbol 74xx:74LS74
Connections:
- new net GND: U?.7 (GND), U?.7 (GND)
- new net VCC: U?.14 (VCC), U?.14 (VCC)
Changed lines of the file:
@@
 F1 "ps3_digital.sch" 50
 $EndSheet
+$Comp
+L 74xx_IEEE:74LS266 U?
+U 4 1 5E9AE710
+P 10200 3050
+AR Path="/5E812EB7/5E9AE710" Ref="U?"  Part="4"
+AR Path="/5E9AE710" Ref="U?"  Part="4"
+F 0 "U?" H 10200 3516 50  0000 C CNN
+F 1 "74LS266" H 10200 3425 50  0000 C CNN
+F 2 "" H 10200 3050 50  0001 C CNN
+F 3 "" H 10200 3050 50  0001 C CNN
+	4    10200 3050
+	1    0    0    -1
+$EndComp
+$Comp
+L 74xx_IEEE:74LS266 U?
+U 3 1 5E9AE716
+P 10200 2200
+AR Path="/5E812EB7/5E9AE716" Ref="U?"  Part="3"
+AR Path="/5E9AE716" Ref="U?"  Part="3"
+F 0 "U?" H 10200 2666 50  0000 C CNN
+F 1 "74LS266" H 10200 2575 50  0000 C CNN
+F 2 "" H 10200 2200 50  0001 C CNN
+F 3 "" H 10200 2200 50  0001 C CNN
+	3    10200 2200
+	1    0    0    -1
+$EndComp
+$Comp
+L 74xx:74LS08 U?
+U 1 1 5E9AE71C
+P 10000 1400
+AR Path="/5E812EB7/5E9AE71C" Ref="U?"  Part="1"
+AR Path="/5E9AE71C" Ref="U?"  Part="1"
+F 0 "U?" H 10000 1725 50  0000 C CNN
+F 1 "74LS08" H 10000 1634 50  0000 C CNN
+F 2 "" H 10000 1400 50  0001 C CNN
+F 3 "http://www.ti.com/lit/gpn/sn74LS08" H 10000 1400 50  0001 C CNN
+	1    10000 1400
+	1    0    0    -1
+$EndComp
+$Comp
+L 74xx:74LS08 U?
+U 1 1 5E9AE722
+P 9100 1400
+AR Path="/5E812EB7/5E9AE722" Ref="U?"  Part="1"
+AR Path="/5E9AE722" Ref="U?"  Part="1"
+F 0 "U?" H 9100 1725 50  0000 C CNN
+F 1 "74LS08" H 9100 1634 50  0000 C CNN
+F 2 "" H 9100 1400 50  0001 C CNN
+F 3 "http://www.ti.com/lit/gpn/sn74LS08" H 9100 1400 50  0001 C CNN
+	1    9100 1400
+	1    0    0    -1
+$EndComp
+$Comp
+L 74xx:74LS32 U?
+U 4 1 5E9AE728
+P 5800 1900
+AR Path="/5E812EB7/5E9AE728" Ref="U?"  Part="4"
+AR Path="/5E9AE728" Ref="U?"  Part="4"
+F 0 "U?" H 5800 2225 50  0000 C CNN
+F 1 "74LS32" H 5800 2134 50  0000 C CNN
+F 2 "" H 5800 1900 50  0001 C CNN
+F 3 "http://www.ti.com/lit/gpn/sn74LS32" H 5800 1900 50  0001 C CNN
+	4    5800 1900
+	1    0    0    -1
+$EndComp
+$Comp
+L 74xx:74LS32 U?
+U 3 1 5E9AE72E
+P 6600 3200
+AR Path="/5E812EB7/5E9AE72E" Ref="U?"  Part="3"
+AR Path="/5E9AE72E" Ref="U?"  Part="3"
+F 0 "U?" H 6600 3525 50  0000 C CNN
+F 1 "74LS32" H 6600 3434 50  0000 C CNN
+F 2 "" H 6600 3200 50  0001 C CNN
+F 3 "http://www.ti.com/lit/gpn/sn74LS32" H 6600 3200 50  0001 C CNN
+	3    6600 3200
+	1    0    0    -1
+$EndComp
+$Comp
+L 74xx:74LS32 U?
+U 2 1 5E9AE734
+P 6550 2600
+AR Path="/5E812EB7/5E9AE734" Ref="U?"  Part="2"
+AR Path="/5E9AE734" Ref="U?"  Part="2"
+F 0 "U?" H 6550 2925 50  0000 C CNN
+F 1 "74LS32" H 6550 2834 50  0000 C CNN
+F 2 "" H 6550 2600 50  0001 C CNN
+F 3 "http://www.ti.com/lit/gpn/sn74LS32" H 6550 2600 50  0001 C CNN
+	2    6550 2600
+	1    0    0    -1
+$EndComp
+$Comp
+L 74xx:74LS32 U?
+U 3 1 5E9AE73A
+P 5850 3200
+AR Path="/5E812EB7/5E9AE73A" Ref="U?"  Part="3"
+AR Path="/5E9AE73A" Ref="U?"  Part="3"
+F 0 "U?" H 5850 3525 50  0000 C CNN
+F 1 "74LS32" H 5850 3434 50  0000 C CNN
+F 2 "" H 5850 3200 50  0001 C CNN
+F 3 "http://www.ti.com/lit/gpn/sn74LS32" H 5850 3200 50  0001 C CNN
+	3    5850 3200
+	1    0    0    -1
+$EndComp
+$Comp
+L 74xx:74LS32 U?
+U 2 1 5E9AE740
+P 5800 2600
+AR Path="/5E812EB7/5E9AE740" Ref="U?"  Part="2"
+AR Path="/5E9AE740" Ref="U?"  Part="2"
+F 0 "U?" H 5800 2925 50  0000 C CNN
+F 1 "74LS32" H 5800 2834 50  0000 C CNN
+F 2 "" H 5800 2600 50  0001 C CNN
+F 3 "http://www.ti.com/lit/gpn/sn74LS32" H 5800 2600 50  0001 C CNN
+	2    5800 2600
+	1    0    0    -1
+$EndComp
+$Comp
+L 74xx:74LS04 U?
+U 5 1 5E9AE746
+P 9150 2600
+AR Path="/5E812EB7/5E9AE746" Ref="U?"  Part="5"
+AR Path="/5E9AE746" Ref="U?"  Part="5"
+F 0 "U?" H 9150 2917 50  0000 C CNN
+F 1 "74LS04" H 9150 2826 50  0000 C CNN
+F 2 "" H 9150 2600 50  0001 C CNN
+F 3 "http://www.ti.com/lit/gpn/sn74LS04" H 9150 2600 50  0001 C CNN
+	5    9150 2600
+	1    0    0    -1
+$EndComp
+$Comp
+L 74xx:74LS04 U?
+U 6 1 5E9AE74C
+P 8350 3150
+AR Path="/5E812EB7/5E9AE74C" Ref="U?"  Part="6"
+AR Path="/5E9AE74C" Ref="U?"  Part="6"
+F 0 "U?" H 8350 3467 50  0000 C CNN
+F 1 "74LS04" H 8350 3376 50  0000 C CNN
+F 2 "" H 8350 3150 50  0001 C CNN
+F 3 "http://www.ti.com/lit/gpn/sn74LS04" H 8350 3150 50  0001 C CNN
+	6    8350 3150
+	1    0    0    -1
+$EndComp
+$Comp
+L 74xx:74LS04 U?
+U 5 1 5E9AE752
+P 8300 2600
+AR Path="/5E812EB7/5E9AE752" Ref="U?"  Part="5"
+AR Path="/5E9AE752" Ref="U?"  Part="5"
+F 0 "U?" H 8300 2917 50  0000 C CNN
+F 1 "74LS04" H 8300 2826 50  0000 C CNN
+F 2 "" H 8300 2600 50  0001 C CNN
+F 3 "http://www.ti.com/lit/gpn/sn74LS04" H 8300 2600 50  0001 C CNN
+	5    8300 2600
+	1    0    0    -1
+$EndComp
+$Comp
+L 74xx:74LS04 U?
+U 4 1 5E9AE758
+P 8300 2000
+AR Path="/5E812EB7/5E9AE758" Ref="U?"  Part="4"
+AR Path="/5E9AE758" Ref="U?"  Part="4"
+F 0 "U?" H 8300 2317 50  0000 C CNN
+F 1 "74LS04" H 8300 2226 50  0000 C CNN
+F 2 "" H 8300 2000 50  0001 C CNN
+F 3 "http://www.ti.com/lit/gpn/sn74LS04" H 8300 2000 50  0001 C CNN
+	4    8300 2000
+	1    0    0    -1
+$EndComp
+$Comp
+L 74xx:74LS04 U?
+U 2 1 5E9AE75E
+P 8300 1350
+AR Path="/5E812EB7/5E9AE75E" Ref="U?"  Part="2"
+AR Path="/5E9AE75E" Ref="U?"  Part="2"
+F 0 "U?" H 8300 1667 50  0000 C CNN
+F 1 "74LS04" H 8300 1576 50  0000 C CNN
+F 2 "" H 8300 1350 50  0001 C CNN
+F 3 "http://www.ti.com/lit/gpn/sn74LS04" H 8300 1350 50  0001 C CNN
+	2    8300 1350
+	1    0    0    -1
+$EndComp
+$Comp
+L 74xx:74LS00 U?
+U 2 1 5E9AE764
+P 7550 2650
+AR Path="/5E812EB7/5E9AE764" Ref="U?"  Part="2"
+AR Path="/5E9AE764" Ref="U?"  Part="2"
+F 0 "U?" H 7550 2975 50  0000 C CNN
+F 1 "74LS00" H 7550 2884 50  0000 C CNN
+F 2 "" H 7550 2650 50  0001 C CNN
+F 3 "http://www.ti.com/lit/gpn/sn74ls00" H 7550 2650 50  0001 C CNN
+	2    7550 2650
+	1    0    0    -1
+$EndComp
+$Comp
+L 74xx:74LS74 U?
+U 2 1 5E9AE76A
+P 7600 1950
+AR Path="/5E812EB7/5E9AE76A" Ref="U?"  Part="2"
+AR Path="/5E9AE76A" Ref="U?"  Part="2"
+F 0 "U?" H 7600 2431 50  0000 C CNN
+F 1 "74LS74" H 7600 2340 50  0000 C CNN
+F 2 "" H 7600 1950 50  0001 C CNN
+F 3 "74xx/74hc_hct74.pdf" H 7600 1950 50  0001 C CNN
+	2    7600 1950
+	1    0    0    -1
+$EndComp
+$Comp
+L 74xx:74LS74 U?
+U 2 1 5E9AE770
+P 6750 1950
+AR Path="/5E812EB7/5E9AE770" Ref="U?"  Part="2"
+AR Path="/5E9AE770" Ref="U?"  Part="2"
+F 0 "U?" H 6750 2431 50  0000 C CNN
+F 1 "74LS74" H 6750 2340 50  0000 C CNN
+F 2 "" H 6750 1950 50  0001 C CNN
+F 3 "74xx/74hc_hct74.pdf" H 6750 1950 50  0001 C CNN
+	2    6750 1950
+	1    0    0    -1
+$EndComp
 $EndSCHEMATC
