File: voicecard.sch (KiCad schematic (older format))
At the start: 23 parts

Commit message: WIP
Parts:
- removed C?: CP, symbol Device:CP
- removed R? (x20): R, symbol Device:R
- removed U? (x2): AS3340, symbol Audio:AS3340
- added C11, C12: 10uF, symbol Device:CP_Small
- added C26: 1nF, symbol Device:C_Small
- added D1, D2, D3, D4: 1N4148, Diode_THT:D_DO-35_SOD27_P7.62mm_Horizontal, symbol Diode:1N4148
- added J1: Conn_01x50_Male, symbol Connector:Conn_01x50_Male
- added Q1, Q2: BF244C, Package_TO_SOT_THT:TO-92_Inline, symbol Transistor_FET:BF244C
- added Q3: 3, Package_TO_SOT_THT:TO-92_Inline, symbol Transistor_FET:BF244C
- added Q4, Q5, Q6, Q8, Q9: BC212L, Package_TO_SOT_THT:TO-92L_Inline_Wide, symbol Device:Q_PNP_BCE
- added R108: 332k, symbol Device:R
- added R109, R110, R118: 1M, symbol Device:R
- added R113, R114, R117: 100k, symbol Device:R
- added R115: 470, symbol Device:R
- added R116: 1M5, symbol Device:R
- added RV4: 100k, symbol Device:R_POT_TRIM_US
- added RV5: 22k, symbol Device:R_POT_TRIM_US
- added U1, U4: AS3340, symbol Audio:AS3340
- added U10, U5, U8: LM13600, symbol Amplifier_Operational:LM13600
- added U11, U9: TL072, symbol Amplifier_Operational:TL072
- added U12, U13: AS3310, symbol Audio:AS3310
- added U2, U3: 4016, symbol 4xxx:4016
- added U6: CA3080, symbol Amplifier_Operational:CA3080
- added U7: LM741, symbol Amplifier_Operational:LM741
Connections:
- net +15V: now also C12.1, J1.21 (Pin_21), J1.22 (Pin_22), R108.1, RV4.3, U1.16 (VCC)
- new net: R110.1, RV4.2
- new net: R109.1, RV5.2
- new net: C26.1, U1.11 (CAP)
- new net -15V: C11.2, J1.25 (Pin_25), J1.26 (Pin_26), RV4.1
- new net -5V: J1.14 (Pin_14), U1.3 (VEE)
- new net ADSR-CONT: J1.40 (Pin_40)
- new net ADSR-ON-OFF: J1.37 (Pin_37)
- new net ADSR_VCA_A1: J1.43 (Pin_43)
- new net ADSR_VCA_D1: J1.44 (Pin_44)
- new net ADSR_VCA_R1: J1.46 (Pin_46)
- new net ADSR_VCA_S1: J1.45 (Pin_45)
- new net CV_OSC1: R108.2, R109.2, R110.2, R113.1, R114.1, R115.2, R116.1, R117.1, R118.1, U1.15 (VFCI)
- new net GATE: J1.42 (Pin_42)
- new net GND: C11.1, C12.2, C26.2, J1.23 (Pin_23), J1.24 (Pin_24), J1.32 (Pin_32), J1.34 (Pin_34), J1.36 (Pin_36), R115.1, RV5.1, U1.12 (GND)
- new net HF_TRACK: RV5.3, U1.7 (VHFT)
- new net KEYBOARD_PITCH: J1.3 (Pin_3), R117.2
- new net NOISE: J1.33 (Pin_33)
- new net O: J1.29 (Pin_29)
- new net OUTPUT: J1.35 (Pin_35)
- new net PITCH_BEND: J1.1 (Pin_1), R118.2
- new net SAW-1: J1.8 (Pin_8)
- new net SAW-2: J1.11 (Pin_11)
- new net SQR-1: J1.6 (Pin_6)
- new net SQR-2: J1.9 (Pin_9)
- new net SYNC: J1.15 (Pin_15)
- new net TRANSPOSE: J1.13 (Pin_13), R113.2
- new net TRI-1: J1.7 (Pin_7)
- new net TRI-2: J1.10 (Pin_10)
- new net VCA_ADSR_TRACK: J1.41 (Pin_41)
- new net VCF_ADSR_TRACK: J1.38 (Pin_38)
- new net VCF_FREQ: J1.28 (Pin_28)
- new net VCF_PITCH_TRACK: J1.31 (Pin_31)
- new net VCF_SWEEP_A2: J1.47 (Pin_47)
- new net VCF_SWEEP_ADSR: J1.27 (Pin_27)
- new net VCF_SWEEP_D2: J1.48 (Pin_48)
- new net VCF_SWEEP_DEPTH: J1.30 (Pin_30)
- new net VCF_SWEEP_R2: J1.50 (Pin_50)
- new net VCF_SWEEP_S2: J1.49 (Pin_49)
- new net VCO1-MOD: J1.17 (Pin_17)
- new net VCO1-TUNE: J1.4 (Pin_4), R116.2
- new net VCO2-MOD: J1.18 (Pin_18)
- new net VCO2-TUNE: J1.12 (Pin_12)
- new net VIBRATO: J1.16 (Pin_16), R114.2
- new net VOL1: J1.19 (Pin_19)
- new net VOL2: J1.20 (Pin_20)
- new net ~ADSR-CONT: J1.39 (Pin_39)
- no-connect marks 0 -> 2

Commit message: Voice Card
Parts:
- added C10: 220nF, symbol Device:C_Small
- added C13, C15, C19, C24, C27 (x2), C30, C31: 10nF, symbol Device:C_Small
- added C15, C16, C21, C22, C29, C?: 1uF, symbol Device:CP_Small
- added C18: 1nF, symbol Device:C_Small
- added C23: 220p, symbol Device:C_Small
- added C25 (x2): 100nF, symbol Device:C_Small
- added Q7: BC212L, Package_TO_SOT_THT:TO-92L_Inline_Wide, symbol Device:Q_PNP_BCE
- added R100, R105, R119, R51, R74, R85, R88, RR87: 10k, symbol Device:R
- added R101, R71, R82: 470, symbol Device:R
- added R103 (x2): 1k82, symbol Device:R
- added R104, R111, R78, R79, R84: 1M, symbol Device:R
- added R106, R93, R99, RR86: 22k, symbol Device:R
- added R107, R87: 5k6, symbol Device:R
- added R112, R75, R76: 100k, symbol Device:R
- added R48, R52, R89, R92: 2k2, symbol Device:R
- added R49: 1k, symbol Device:R
- added R62, RR102, RR47: 47k, symbol Device:R
- added R70: 332k, symbol Device:R
- added R72, R73, R94, R95, R96: 68k, symbol Device:R
- added R77: 1M5, symbol Device:R
- added R90, R91: 15k, symbol Device:R
- added RV6, RV9: 10k, symbol Device:R_POT_TRIM
- added RV7: 100k, symbol Device:R_POT_TRIM_US
- added RV8: 22k, symbol Device:R_POT_TRIM_US
Connections:
- net +15V: now also U4.16 (VCC), C15.2, C?.2, R100.1, R104.1, R70.1, R84.1, R88.1, R90.2, R91.2, RV7.3
- net -15V: now also Q8.2 (C), Q7.2 (C), RV7.1
- net -5V: now also Q9.2 (C), U4.3 (VEE), C16.2, C29.2, R107.1, R87.1, RV6.1, RV6.2, RV9.1, RV9.2
- net GND: now also U4.12 (GND), C13.2, C15.1, C15.2, C16.1, C18.2, C19.2, C24.2, C25.2, C25.2, C27.2, C27.2, C29.1, C30.2, C31.2, C?.1, R103.2, R103.2, R105.1, R48.1, R49.1, R51.1, R52.2, R85.1, R89.2, R92.1, RV8.1; no longer R115.1
- net KEYBOARD_PITCH: now also R112.2
- net NOISE: now also R62.2
- net PITCH_BEND: now also R111.2
- net SAW-2: now also U2.5, U3.6
- net SQR-1: now also U2.13
- net SQR-2: now also U3.12
- net SYNC: now also U2.6
- net TRANSPOSE: now also R76.2
- net TRI-2: now also U2.12, U3.5
- net VCO1-MOD: now also R119.2
- net VCO2-MOD: now also R74.2
- net VCO2-TUNE: now also R77.2
- net VIBRATO: now also R75.2
- net VOL1: now also R73.2
- net VOL2: now also R72.2
- net VCO1_SCALE1: now reaches U1.1 (SCALE1)
- net VCO1_SCALE1: now also R106.1
- net VCO1_TRI_OUT: now reaches U1.10 (VTO)
- net VCO1_TRI_OUT: now also Q8.1 (B), Q9.3 (E)
- net at U1.13 (VLFI): now also R101.1, R104.2
- net at U1.14 (VS): now also C27.1, R103.1
- net VCO1_SCALE2: now reaches U1.2 (SCALE2)
- net VCO1_SCALE2: now also R107.2
- net VCO1_SQR_OUT: now reaches U1.4 (VP)
- net VCO1_SQR_OUT: now also R105.2, R96.1
- net VCO1_PWM_IN: now reaches U1.5 (VPWM)
- net VCO1_PWM_IN: now also C30.1, R119.1
- net VCO1_SAW_OUT: now reaches U1.8 (VSO)
- net VCO1_SAW_OUT: now also U2.4
- net VCO1_SYNC: now reaches U1.9 (VSSI)
- net VCO1_SYNC: now also C25.1, RR102.2
- net VCO2_SCALE1: now reaches U4.1 (SCALE1)
- net VCO2_SCALE1: now also RR86.1
- net VCO2_TRI_OUT: now reaches U4.10 (VTO)
- net VCO2_TRI_OUT: now also Q7.1 (B)
- net at U4.11 (CAP): now also C18.1
- net at U4.13 (VLFI): now also R82.1, R84.2
- net at U4.14 (VS): now also C27.1, R103.1
- net VCO2_CV: now reaches U4.15 (VFCI)
- net VCO2_CV: now also R111.1, R112.1, R70.2, R71.2, R75.1, R76.1, R77.1, R78.2, R79.2
- net VCO2_SCALE2: now reaches U4.2 (SCALE2)
- net VCO2_SCALE2: now also R87.2
- net VCO2_SQR_OUT: now reaches U4.4 (VP)
- net VCO2_SQR_OUT: now also R85.2, R95.1
- net VCO2_PWM_IN: now reaches U4.5 (VPWM)
- net VCO2_PWM_IN: now also C15.1, R74.1
- net HF_TRACK_VCO2: now reaches U4.7 (VHFT)
- net HF_TRACK_VCO2: now also RV8.3
- net at U4.8 (VSO): now also R94.2
- net VCO2_SYNC: now reaches U4.9 (VSSI)
- net VCO2_SYNC: now also C25.1
- net at U2.1: now also R96.2
- net VCO1_OUT: now reaches U2.2
- net VCO1_OUT: now also U2.11, U2.3, C22.1
- net VCO2_SAW_OUT: now reaches U2.8
- net VCO2_SAW_OUT: now also U3.8, R94.1
- net at U2.9: now also C23.1
- net at U2.10: now also R99.2
- net VCO2_OUT: now reaches U3.10
- net VCO2_OUT: now also U3.3, U3.9, C21.1
- net at U3.11: now also R95.2
- net at U3.4: now also R93.2
- net at U5.12: now also U5.5, C10.2, R51.2
- net at U5.13 (-): now also R89.1
- net at U5.14 (+): now also C22.2, R92.2
- net at U5.15 (DIODE_BIAS): now also R90.1
- net at U5.16: now also R73.1
- net at U5.1: now also R72.1
- net at U5.2 (DIODE_BIAS): now also R91.1
- net at U5.3 (+): now also C21.2, R48.2
- net at U5.4 (-): now also R52.1
- net at Q8.3 (E): now also R100.2, R99.1
- net at Q9.1 (B): now also RR102.1, RR87.2
- net CV_OSC1 renamed VCO1_CV
- net HF_TRACK renamed HF_TRACK_VCO1
- new net: C31.1, R115.1
- new net: R79.1, RV7.2
- new net: R78.1, RV8.2
- new net: C13.1, R71.1
- new net: R106.2, RV9.3
- new net: RR86.2, RV6.3
- new net: C23.2, RR87.1
- new net: Q7.3 (E), R88.2, R93.1
- new net: C19.1, R82.2
- new net: C24.1, R101.2
- new net: C10.1, RR47.2
- new net: R49.2, R62.1, RR47.1
Other:
- note added: "VCO1 CV"
- note added: "VCO1 SCALE"
- note added: "VCO1 SYNC"
- moved on the sheet: C26, D1, D2, D3, D4, Q1, Q2, Q3, Q4, Q5, Q6, Q8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

Commit message: Voice Card ...
Parts:
- removed D1, D4: 1N4148, Diode_THT:D_DO-35_SOD27_P7.62mm_Horizontal, symbol Diode:1N4148
- removed Q1: BF244C, Package_TO_SOT_THT:TO-92_Inline, symbol Transistor_FET:BF244C
- added C1, C4: 22nF, symbol Device:C_Small
- added C5: 3.3nF, symbol Device:C_Small
- added C7, C9, C?: 1nF, symbol Device:C_Small
- added C8: 220nF, symbol Device:C_Small
- added D2: 1N4148, Diode_THT:D_DO-35_SOD27_P7.62mm_Horizontal, symbol Diode:1N4148
- added D4: 1N4148, symbol Device:D
- added Q2: BF244C, Package_TO_SOT_THT:TO-92_Inline, symbol Transistor_FET:BF244C
- added R10, R11, R13, R14, R38, R42, R45, R54, R56, R58: 100k, symbol Device:R
- added R12, R63, R8: 3M3, symbol Device:R
- added R15, R53, R61, R9: 1M, symbol Device:R
- added R16, R17, R39, R50, R55, R59, R66: 1k, symbol Device:R
- added R19, R6: 6k6, symbol Device:R
- added R21, R31: 66, symbol Device:R
- added R27: 16k, symbol Device:R
- added R28, R46, R?: 22k, symbol Device:R
- added R33, R60, R68, R81: 47k, symbol Device:R
- added R40, R41, R43, R7: 10k, symbol Device:R
- added R44: 15k, symbol Device:R
- added R57: 220, symbol Device:R
- added R64: 750k, symbol Device:R
- added R65: 1k8, symbol Device:R
- added R67: 120k, symbol Device:R
- added R68: 150k, symbol Device:R
- added R8, R?: 820, symbol Device:R
- added R80: 18k, symbol Device:R
- added RV1, RV2: 100k, symbol Device:R_POT_TRIM
- added RV3: 22k, symbol Device:R_POT_TRIM
- Q3: value 3 -> BF244C
- renumbered D2 to D1, Q2 to Q1, RR102 to R102, RR47 to R47, RR86 to R86, RR87 to R87
Connections:
- net +15V: now also U10.11 (V+), U11.8 (V+), U12.11 (VCC), U5.11 (V+), U6.7 (V+), U7.7 (V+), U8.11 (V+), U9.8 (V+), R33.2, R44.1, R63.2, RV1.3, RV2.1
- net -15V: now also U10.6 (V-), U11.4 (V-), U5.6 (V-), U6.4 (V-), U7.4 (V-), U8.6 (V-), U9.4 (V-), R12.2, R8.2, R8.2, RV1.1, RV2.3
- net ADSR-ON-OFF: now also Q4.3 (E), R38.2
- net GATE: now also U12.4 (GATE), C5.1, R7.1
- net GND: now also Q5.2 (C), U11.3 (+), U11.5 (+), U12.7 (PGND), U13.7 (PGND), C1.1, C4.1, C7.1, C9.1, D4.2 (A), R16.1, R17.1, R21.1, R31.1, R39.1, R41.1, R43.1, R50.1, R55.1, R59.1, R65.1, R66.1, R7.2
- net KEYBOARD_PITCH: now also U3.1, R10.2, R14.2
- net O: now also R61.2
- net OUTPUT: now also R40.2
- net VCA_ADSR_TRACK: now also D2.1 (K)
- net VCF_ADSR_TRACK: now also D3.1 (K)
- net VCF_FREQ: now also R68.2
- net VCF_PITCH_TRACK: now also U3.13
- net VCF_SWEEP_ADSR: now also RV3.1
- net VCF_SWEEP_DEPTH: now also R67.2
- net ~ADSR-CONT: now also R38.1
- net VCA_ADSR_GND: now reaches U13.14 (GND)
- net VCA_ADSR_GND: now also R31.2, R6.1
- net VCA_ADSR_CCOMP: now reaches U13.8 (CCOMP)
- net VCA_ADSR_CCOMP: now also C1.2
- net VCF_ADSR_GND: now reaches U12.14 (GND)
- net VCF_ADSR_GND: now also R19.1, R21.2
- net VCF_ADSR_TRIG: now reaches U12.5 (TRIG)
- net VCF_ADSR_TRIG: now also C5.2
- net at U12.6 (VEE): now also R8.1
- net VCF_ADSR_CCOMP: now reaches U12.8 (CCOMP)
- net VCF_ADSR_CCOMP: now also C4.2
- net at U3.2: now also R81.1
- net at U8.12: now also U10.13 (-), R50.2, R53.2
- net at U8.13 (-): now also R59.2
- net at U8.14 (+): now also R54.1, R55.2
- net at U8.16: now also R61.1
- net at U8.1: now also R27.2
- net at U8.2 (DIODE_BIAS): now also R44.2
- net at U8.3 (+): now also R28.1, R41.2, R42.2
- net at U8.4 (-): now also R43.2
- net at U8.5: now also R40.1
- net at U10.12: now also U9.5 (+), C9.2
- net at U10.14 (+): now also R47.1, R49.2, R62.1, R58.2
- net at U10.16: now also R46.1
- net at U10.1: now also R?.1
- net at U10.3 (+): now also R16.2
- net at U10.4 (-): now also R17.2, R45.1
- net at U10.5: now also U9.3 (+), C7.2
- net at U6.2 (-): now also R56.2, R57.2
- net at U6.3 (+): now also R57.1
- net at U6.5 (BIAS): now also R80.2
- net at U6.6: now also Q5.1 (B), R60.1, R66.2, R67.1, R68.1, R68.1, R81.2
- net at U7.2 (-): now also Q6.3 (E), U7.6, D4.1 (K)
- net at U7.3 (+): now also Q5.3 (E), R63.1
- net at U9.1: now also U9.2 (-), C8.2, R58.1
- net at U9.6 (-): now also U9.7, R45.2, R53.1, R54.2
- net at U11.1: now also Q2.3 (S), R11.1, R6.2, R9.2
- net at U11.2 (-): now also Q2.1 (D), R10.1, R11.2, R8.1
- net at U11.6 (-): now also Q3.1 (D), R12.1, R13.2, R14.1
- net at U11.7: now also Q3.3 (S), R13.1, R15.2, R19.2
- net at Q3.2 (G): now also D3.2 (A), R15.1
- net at Q4.1 (B): now also R33.1, R39.2
- net at Q4.2 (C): now also R27.1
- net at Q6.1 (B): now also R64.1, R65.2
- net at Q6.2 (C): now also R46.2, R?.2
- new net: C8.1, R28.2
- new net: R64.2, RV2.2
- new net: R56.1, R60.2
- new net: R80.1, RV3.2, RV3.3
- new net: R42.1, RV1.2
- new net: D2.2 (A), Q2.2 (G), R9.1
- no-connect marks 2 -> 6
Other:
- note added: "VCF CONTROL"
- moved on the sheet: C11, C12, D1, D3, Q1, Q3, Q4, Q5, Q6, R62, U10B, U10C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

Commit message: Voice Card done
Parts:
- removed C?: 1nF, symbol Device:C_Small
- removed R?: 820, symbol Device:R
- added C2: 3.3nF, symbol Device:C_Small
- added C3, C6: 47nF, symbol Device:C_Small
- added R1: 18k, symbol Device:R
- added R2, R28: 47k, symbol Device:R
- added R20, R22, R23, R30, R32, R34: 470, symbol Device:R
- added R24, R25, R26, R35, R36, R37: 30k, symbol Device:R
- added R3: 820, symbol Device:R
- added R4: 1M, symbol Device:R
- gave numbers to parts that had none: 2
Connections:
- net ADSR_VCA_A1 is gone; now on net VCA_ADSR_A1: J1.43 (Pin_43)
- net ADSR_VCA_D1 is gone; now on net VCA_ADSR_D1: J1.44 (Pin_44)
- net ADSR_VCA_R1 is gone; now on net VCA_ADSR_R1: J1.46 (Pin_46)
- net ADSR_VCA_S1 is gone; now on net VCA_ADSR_S1: J1.45 (Pin_45)
- net +15V: now also U13.11 (VCC), U2.14 (VDD), U3.14 (VDD)
- net -15V: now also R3.2
- net ADSR-CONT: now also D1.1 (K)
- net ADSR-ON-OFF: now also R1.2
- net GATE: now also U13.4 (GATE), C2.1
- net GND: now also U2.7 (VSS), U3.7 (VSS), C3.1, C6.1, R20.2, R22.2, R23.2, R30.2, R32.2, R34.2
- net VCF_SWEEP_A2: now also R26.2
- net VCF_SWEEP_D2: now also R25.2
- net VCF_SWEEP_R2: now also R24.2
- net VCF_SWEEP_S2: now also U12.9 (VCS)
- net at U13.1 (CAP): now also C3.2
- net at U13.10 (IIN): now also R2.1
- net VCA_ADSR_D1: now reaches U13.12 (VCD)
- net VCA_ADSR_R1: now reaches U13.13 (VCR)
- net VCA_ADSR_A1: now reaches U13.15 (VCA)
- net at U13.2 (ENVOUT): now also Q1.1 (D), R2.2, R4.2
- net VCA_ADSR_TRIG: now reaches U13.5 (TRIG)
- net VCA_ADSR_TRIG: now also C2.2
- net at U13.6 (VEE): now also R3.1
- net VCA_ADSR_S1: now reaches U13.9 (VCS)
- net at U12.1 (CAP): now also C6.2
- net at U12.10 (IIN): now also R28.1
- net VCF_ADSR_D: now reaches U12.12 (VCD)
- net VCF_ADSR_D: now also R23.1, R25.1
- net VCF_ADSR_R: now reaches U12.13 (VCR)
- net VCF_ADSR_R: now also R22.1, R24.1
- net VCF_ADSR_A: now reaches U12.15 (VCA)
- net VCF_ADSR_A: now also R20.1, R26.1
- net at U12.2 (ENVOUT): now also R56.1, R60.2, R28.2
- net at Q1.2 (G): now also D1.2 (A), R4.1
- net at Q1.3 (S): now also R1.1
- new net VCA_ADSR_A: R30.1, R37.1
- new net VCA_ADSR_D: R34.1, R36.1
- new net VCA_ADSR_R: R32.1, R35.1
- new net VCA_SWEEP_A2: R37.2
- new net VCA_SWEEP_D2: R36.2
- new net VCA_SWEEP_R2: R35.2
- no-connect marks 6 -> 18
Other:
- moved on the sheet: C1, C5, D1, D2, Q1, Q2, R10, R11, R31, R6, R7, R8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
